File: current_conditioner.kicad_pcb (KiCad board)
At the start: 2 copper layers, 36.8 x 56.8 mm, 21 parts, among them J1 RJ45, P1 CON, P2 gnd_ref, U1 AD8422, U2 AD8609

Commit message: Did PCB layout
Parts:
- moved JP1 22.9 mm to (68.6, 47.6), turned to 90 degrees
- moved C2 17.6 mm to (48.3, 54.0)
- moved R4 10.9 mm to (54.6, 57.8)
- moved C1 8.28 mm to (48.3, 57.8), turned to 180 degrees
- moved RP1 7.73 mm to (48.9, 47.0), turned to 90 degrees
- moved R5 4.02 mm to (61.0, 54.0)
- moved R2 3.17 mm to (57.8, 59.1), turned to 270 degrees
- moved U2 1.80 mm to (57.8, 48.9)
- moved R3 1.80 mm to (54.6, 54.6)
- moved U1 1.42 mm to (57.8, 64.8)
- moved P2 0.90 mm to (66.0, 56.5)
- moved R1 0.90 mm to (57.8, 69.8)
Changed lines of the file:
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@@
     (pad_to_mask_clearance 0)
     (aux_axis_origin 0 0)
-    (visible_elements 7FFFFF7F)
+    (visible_elements 7FFFFB7F)
     (pcbplotparams
       (layerselection 283148289)
@@
   )
   (module SO8E (layer F.Cu)
-    (at 57.15 63.5)
+    (at 57.785 64.77)
     (descr "module CMS SOJ 8 pins etroit")
     (tags "CMS SOJ")
@@
   )
   (module SO14E (layer F.Cu)
-    (at 59.055 47.625)
+    (at 57.785 48.895)
     (descr "module CMS SOJ 14 pins etroit")
     (tags "CMS SOJ")
@@
   )
   (module SM1206POL_VIS (layer F.Cu)
-    (at 64.135 61.595)
+    (at 48.26 53.975)
     (attr smd)
     (fp_text reference C2 (at 0 -1.8288) (layer F.SilkS)
@@
   )
   (module SM0603_VIS (layer F.Cu)
-    (at 59.69 57.785)
+    (at 60.96 53.975)
     (attr smd)
     (fp_text reference R5 (at 0 -1.016) (layer F.SilkS)
@@
   )
   (module SM0603_VIS (layer F.Cu)
-    (at 48.26 48.895)
+    (at 54.61 57.785)
     (attr smd)
     (fp_text reference R4 (at 0 -1.016) (layer F.SilkS)
@@
   )
   (module SM0603_VIS (layer F.Cu)
-    (at 55.88 53.34 180)
+    (at 54.61 54.61 180)
     (attr smd)
     (fp_text reference R3 (at 0 -1.016 180) (layer F.SilkS)
@@
   )
   (module SM0603_VIS (layer F.Cu)
-    (at 55.88 56.515 180)
-    (attr smd)
-    (fp_text reference R2 (at 0 -1.016 180) (layer F.SilkS)
-      (effects (font (size 0.508 0.508) (thickness 0.1143)))
-    )
-    (fp_text value 10k (at 0 1.143 180) (layer F.SilkS)
+    (at 57.785 59.055 270)
+    (attr smd)
+    (fp_text reference R2 (at 0 -1.016 270) (layer F.SilkS)
+      (effects (font (size 0.508 0.508) (thickness 0.1143)))
+    )
+    (fp_text value 10k (at 0 1.143 270) (layer F.SilkS)
       (effects (font (size 0.508 0.508) (thickness 0.1143)))
     )
@@
     (fp_line (start 1.143 0.635) (end -1.143 0.635) (layer F.SilkS) (width 0.127))
     (fp_line (start -1.143 0.635) (end -1.143 -0.635) (layer F.SilkS) (width 0.127))
-    (pad 1 smd rect (at -0.762 0 180) (size 0.635 1.143)
+    (pad 1 smd rect (at -0.762 0 270) (size 0.635 1.143)
       (layers F.Cu F.Paste F.Mask)
       (net 13 N-000026)
     )
-    (pad 2 smd rect (at 0.762 0 180) (size 0.635 1.143)
+    (pad 2 smd rect (at 0.762 0 270) (size 0.635 1.143)
       (layers F.Cu F.Paste F.Mask)
       (net 11 N-000024)
@@
   )
   (module SM0603_VIS (layer F.Cu)
-    (at 57.15 69.215)
+    (at 57.785 69.85)
     (attr smd)
     (fp_text reference R1 (at 0 -1.016) (layer F.SilkS)
@@
   )
   (module SM0603_Capa_VIS (layer F.Cu)
-    (at 47.625 66.04)
-    (attr smd)
-    (fp_text reference C1 (at 0 -1.0414) (layer F.SilkS)
+    (at 48.26 57.785 180)
+    (attr smd)
+    (fp_text reference C1 (at 0 -1.0414 180) (layer F.SilkS)
       (effects (font (size 0.508 0.4572) (thickness 0.1143)))
     )
-    (fp_text value 1n (at 0 1.143) (layer F.SilkS)
+    (fp_text value 1n (at 0 1.143 180) (layer F.SilkS)
       (effects (font (size 0.508 0.4572) (thickness 0.1143)))
     )
@@
     (fp_line (start 1.19888 -0.635) (end 1.19888 0.635) (layer F.SilkS) (width 0.11938))
     (fp_line (start -1.19888 0.635) (end -1.19888 -0.635) (layer F.SilkS) (width 0.11938))
-    (pad 1 smd rect (at -0.762 0) (size 0.635 1.143)
+    (pad 1 smd rect (at -0.762 0 180) (size 0.635 1.143)
       (layers F.Cu F.Paste F.Mask)
       (net 3 GND)
     )
-    (pad 2 smd rect (at 0.762 0) (size 0.635 1.143)
+    (pad 2 smd rect (at 0.762 0 180) (size 0.635 1.143)
       (layers F.Cu F.Paste F.Mask)
       (net 1 +5V)
@@
   )
   (module RESARRAY-0612 (layer F.Cu)
-    (at 47.625 54.61)
-    (fp_text reference RP1 (at 0 2) (layer F.SilkS)
+    (at 48.895 46.99 90)
+    (fp_text reference RP1 (at 0 2 90) (layer F.SilkS)
       (effects (font (size 0.7 0.7) (thickness 0.125)))
     )
-    (fp_text value R_PACK4 (at 0 -1.75) (layer F.SilkS)
+    (fp_text value R_PACK4 (at 0 -1.75 90) (layer F.SilkS)
       (effects (font (size 0.7 0.7) (thickness 0.08)))
     )
@@
     (fp_line (start 2 1.25) (end -2 1.25) (layer F.SilkS) (width 0.15))
     (fp_line (start -2 1.25) (end -2 -1.25) (layer F.SilkS) (width 0.15))
-    (pad 1 smd rect (at -1.3 0.7) (size 0.7 0.7)
+    (pad 1 smd rect (at -1.3 0.7 90) (size 0.7 0.7)
       (layers F.Cu F.Paste F.Mask)
       (net 10 N-000023)
     )
-    (pad 2 smd rect (at -0.4 0.7) (size 0.5 0.7)
+    (pad 2 smd rect (at -0.4 0.7 90) (size 0.5 0.7)
       (layers F.Cu F.Paste F.Mask)
       (net 3 GND)
     )
-    (pad 3 smd rect (at 0.4 0.7) (size 0.5 0.7)
-      (layers F.Cu F.Paste F.Mask)
-    )
-    (pad 4 smd rect (at 1.25 0.7) (size 0.7 0.7)
-      (layers F.Cu F.Paste F.Mask)
-    )
-    (pad 5 smd rect (at 1.25 -0.7) (size 0.7 0.7)
-      (layers F.Cu F.Paste F.Mask)
-    )
-    (pad 6 smd rect (at 0.4 -0.7) (size 0.5 0.7)
-      (layers F.Cu F.Paste F.Mask)
-    )
-    (pad 7 smd rect (at -0.4 -0.7) (size 0.5 0.7)
+    (pad 3 smd rect (at 0.4 0.7 90) (size 0.5 0.7)
+      (layers F.Cu F.Paste F.Mask)
+    )
+    (pad 4 smd rect (at 1.25 0.7 90) (size 0.7 0.7)
+      (layers F.Cu F.Paste F.Mask)
+    )
+    (pad 5 smd rect (at 1.25 -0.7 90) (size 0.7 0.7)
+      (layers F.Cu F.Paste F.Mask)
+    )
+    (pad 6 smd rect (at 0.4 -0.7 90) (size 0.5 0.7)
+      (layers F.Cu F.Paste F.Mask)
+    )
+    (pad 7 smd rect (at -0.4 -0.7 90) (size 0.5 0.7)
       (layers F.Cu F.Paste F.Mask)
       (net 7 N-000014)
     )
-    (pad 8 smd rect (at -1.3 -0.7) (size 0.7 0.7)
+    (pad 8 smd rect (at -1.3 -0.7 90) (size 0.7 0.7)
       (layers F.Cu F.Paste F.Mask)
       (net 7 N-000014)
@@
   )
   (module PIN_ARRAY_3X1 (layer F.Cu)
-    (at 49.53 60.325)
+    (at 68.58 47.625 90)
     (descr "Connecteur 3 pins")
     (tags "CONN DEV")
-    (fp_text reference JP1 (at 0.254 -2.159) (layer F.SilkS)
+    (fp_text reference JP1 (at 0.254 -2.159 90) (layer F.SilkS)
       (effects (font (size 1.016 1.016) (thickness 0.1524)))
     )
-    (fp_text value JUMPER3 (at 0 -2.159) (layer F.SilkS) hide
+    (fp_text value JUMPER3 (at 0 -2.159 90) (layer F.SilkS) hide
       (effects (font (size 1.016 1.016) (thickness 0.1524)))
     )
@@
     (fp_line (start 3.81 1.27) (end -3.81 1.27) (layer F.SilkS) (width 0.1524))
     (fp_line (start -1.27 -1.27) (end -1.27 1.27) (layer F.SilkS) (width 0.1524))
-    (pad 1 thru_hole rect (at -2.54 0) (size 1.524 1.524) (drill 1.016)
+    (pad 1 thru_hole rect (at -2.54 0 90) (size 1.524 1.524) (drill 1.016)
       (layers *.Cu *.Mask F.SilkS)
       (net 1 +5V)
     )
-    (pad 2 thru_hole circle (at 0 0) (size 1.524 1.524) (drill 1.016)
+    (pad 2 thru_hole circle (at 0 0 90) (size 1.524 1.524) (drill 1.016)
       (layers *.Cu *.Mask F.SilkS)
       (net 10 N-000023)
     )
-    (pad 3 thru_hole circle (at 2.54 0) (size 1.524 1.524) (drill 1.016)
+    (pad 3 thru_hole circle (at 2.54 0 90) (size 1.524 1.524) (drill 1.016)
       (layers *.Cu *.Mask F.SilkS)
       (net 2 AREF)
@@
   )
   (module PIN_ARRAY_1 (layer F.Cu)
-    (at 65.405 55.88)
+    (at 66.04 56.515)
     (descr "1 pin")
     (tags "CONN DEV")

Commit message: Did some routing
Parts:
- turned RP1 to 270 degrees
Routing:
- net N-000017: track 0.00 -> 21.7 mm
- net GND: track 0.00 -> 13.9 mm
- net N-000014: track 0.00 -> 12.5 mm
- net N-000002: track 0.00 -> 8.87 mm
- net N-000026: track 0.00 -> 8.76 mm
- net N-000027: track 0.00 -> 6.15 mm
- net N-000024: track 0.00 -> 2.55 mm
- net N-000009: track 0.00 -> 2.47 mm
- net N-000001: track 0.00 -> 2.47 mm
- net N-000025: track 0.00 -> 2.34 mm
- net out: track 0.00 -> 2.34 mm
- net N-000015: track 0.00 -> 2.30 mm
Changed lines of the file:
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@@
   (general
     (links 36)
-    (no_connects 36)
+    (no_connects 21)
     (area 38.749999 33.949999 75.650001 90.850001)
     (thickness 1.6)
     (drawings 10)
-    (tracks 0)
+    (tracks 49)
     (zones 0)
     (modules 21)
@@
   )
   (module RESARRAY-0612 (layer F.Cu)
-    (at 48.895 46.99 90)
-    (fp_text reference RP1 (at 0 2 90) (layer F.SilkS)
+    (at 48.895 46.99 270)
+    (fp_text reference RP1 (at 0 2 270) (layer F.SilkS)
       (effects (font (size 0.7 0.7) (thickness 0.125)))
     )
-    (fp_text value R_PACK4 (at 0 -1.75 90) (layer F.SilkS)
+    (fp_text value R_PACK4 (at 0 -1.75 270) (layer F.SilkS)
       (effects (font (size 0.7 0.7) (thickness 0.08)))
     )
@@
     (fp_line (start 2 1.25) (end -2 1.25) (layer F.SilkS) (width 0.15))
     (fp_line (start -2 1.25) (end -2 -1.25) (layer F.SilkS) (width 0.15))
-    (pad 1 smd rect (at -1.3 0.7 90) (size 0.7 0.7)
+    (pad 1 smd rect (at -1.3 0.7 270) (size 0.7 0.7)
       (layers F.Cu F.Paste F.Mask)
       (net 10 N-000023)
     )
-    (pad 2 smd rect (at -0.4 0.7 90) (size 0.5 0.7)
+    (pad 2 smd rect (at -0.4 0.7 270) (size 0.5 0.7)
       (layers F.Cu F.Paste F.Mask)
       (net 3 GND)
     )
-    (pad 3 smd rect (at 0.4 0.7 90) (size 0.5 0.7)
-      (layers F.Cu F.Paste F.Mask)
-    )
-    (pad 4 smd rect (at 1.25 0.7 90) (size 0.7 0.7)
-      (layers F.Cu F.Paste F.Mask)
-    )
-    (pad 5 smd rect (at 1.25 -0.7 90) (size 0.7 0.7)
-      (layers F.Cu F.Paste F.Mask)
-    )
-    (pad 6 smd rect (at 0.4 -0.7 90) (size 0.5 0.7)
-      (layers F.Cu F.Paste F.Mask)
-    )
-    (pad 7 smd rect (at -0.4 -0.7 90) (size 0.5 0.7)
+    (pad 3 smd rect (at 0.4 0.7 270) (size 0.5 0.7)
+      (layers F.Cu F.Paste F.Mask)
+    )
+    (pad 4 smd rect (at 1.25 0.7 270) (size 0.7 0.7)
+      (layers F.Cu F.Paste F.Mask)
+    )
+    (pad 5 smd rect (at 1.25 -0.7 270) (size 0.7 0.7)
+      (layers F.Cu F.Paste F.Mask)
+    )
+    (pad 6 smd rect (at 0.4 -0.7 270) (size 0.5 0.7)
+      (layers F.Cu F.Paste F.Mask)
+    )
+    (pad 7 smd rect (at -0.4 -0.7 270) (size 0.5 0.7)
       (layers F.Cu F.Paste F.Mask)
       (net 7 N-000014)
     )
-    (pad 8 smd rect (at -1.3 -0.7 90) (size 0.7 0.7)
+    (pad 8 smd rect (at -1.3 -0.7 270) (size 0.7 0.7)
       (layers F.Cu F.Paste F.Mask)
       (net 7 N-000014)
@@
   (gr_arc (start 72.2 37.4) (end 72.2 34) (angle 90) (layer Edge.Cuts) (width 0.1))
   (gr_arc (start 42.2 37.4) (end 38.8 37.2) (angle 90) (layer Edge.Cuts) (width 0.1))
+  (segment (start 48.195 48.29) (end 48.15 48.335) (width 0.508) (layer F.Cu) (net 0))
+  (segment (start 57.785 46.355) (end 57.785 44.685) (width 0.508) (layer F.Cu) (net 3))
+  (segment (start 49.58 39.63) (end 49.58 37.65) (width 0.508) (layer F.Cu) (net 3))
+  (segment (start 52.4 42.45) (end 49.58 39.63) (width 0.508) (layer F.Cu) (net 3))
+  (segment (start 55.55 42.45) (end 52.4 42.45) (width 0.508) (layer F.Cu) (net 3))
+  (segment (start 57.785 44.685) (end 55.55 42.45) (width 0.508) (layer F.Cu) (net 3))
+  (segment (start 58.547 69.85) (end 58.547 67.564) (width 0.508) (layer F.Cu) (net 4))
+  (segment (start 58.547 67.564) (end 58.42 67.437) (width 0.508) (layer F.Cu) (net 4))
+  (segment (start 55.88 67.437) (end 55.88 71.655) (width 0.508) (layer F.Cu) (net 5))
+  (segment (start 59.055 72.555) (end 59.055 73.66) (width 0.508) (layer F.Cu) (net 5))
+  (segment (start 58.45 71.95) (end 59.055 72.555) (width 0.508) (layer F.Cu) (net 5))
+  (segment (start 56.175 71.95) (end 58.45 71.95) (width 0.508) (layer F.Cu) (net 5))
+  (segment (start 55.88 71.655) (end 56.175 71.95) (width 0.508) (layer F.Cu) (net 5))
+  (segment (start 57.023 69.85) (end 57.023 67.564) (width 0.508) (layer F.Cu) (net 6))
+  (segment (start 57.023 67.564) (end 57.15 67.437) (width 0.508) (layer F.Cu) (net 6))
+  (segment (start 58.935 47.975) (end 58.935 47.515) (width 0.508) (layer F.Cu) (net 7))
+  (segment (start 51.36 46.59) (end 52.05 47.28) (width 0.508) (layer F.Cu) (net 7))
+  (segment (start 52.05 47.28) (end 52.355 47.28) (width 0.508) (layer F.Cu) (net 7))
+  (segment (start 52.355 47.28) (end 53.05 47.975) (width 0.508) (layer F.Cu) (net 7))
+  (segment (start 53.05 47.975) (end 58.935 47.975) (width 0.508) (layer F.Cu) (net 7))
+  (segment (start 49.595 46.59) (end 51.36 46.59) (width 0.508) (layer F.Cu) (net 7) (status 400000))
+  (segment (start 59.055 47.395) (end 59.055 46.355) (width 0.508) (layer F.Cu) (net 7) (status 800000))
+  (segment (start 58.935 47.515) (end 59.055 47.395) (width 0.508) (layer F.Cu) (net 7))
+  (segment (start 49.595 45.69) (end 49.595 46.59) (width 0.508) (layer F.Cu) (net 7) (status C00000))
+  (segment (start 43.815 45.8343) (end 43.815 48.133) (width 0.508) (layer F.Cu) (net 8))
+  (segment (start 63.65 77.05) (end 62.975 77.05) (width 0.508) (layer F.Cu) (net 9))
+  (segment (start 60.262 67.437) (end 63.65 70.825) (width 0.508) (layer F.Cu) (net 9))
+  (segment (start 63.65 70.825) (end 63.65 77.05) (width 0.508) (layer F.Cu) (net 9))
+  (segment (start 59.69 67.437) (end 60.262 67.437) (width 0.508) (layer F.Cu) (net 9))
+  (segment (start 57.745 78.7) (end 55.245 76.2) (width 0.508) (layer F.Cu) (net 9))
+  (segment (start 61.325 78.7) (end 57.745 78.7) (width 0.508) (layer F.Cu) (net 9))
+  (segment (start 62.975 77.05) (end 61.325 78.7) (width 0.508) (layer F.Cu) (net 9))
+  (segment (start 57.15 62.103) (end 57.15 60.452) (width 0.508) (layer F.Cu) (net 11))
+  (segment (start 57.15 60.452) (end 57.785 59.817) (width 0.508) (layer F.Cu) (net 11))
+  (segment (start 60.198 52.827) (end 60.198 53.975) (width 0.508) (layer F.Cu) (net 12))
+  (segment (start 60.325 52.7) (end 60.198 52.827) (width 0.508) (layer F.Cu) (net 12))
+  (segment (start 60.325 51.689) (end 60.325 52.7) (width 0.508) (layer F.Cu) (net 12))
+  (segment (start 55.372 54.61) (end 57.26 54.61) (width 0.508) (layer F.Cu) (net 13))
+  (segment (start 57.785 55.135) (end 57.785 58.293) (width 0.508) (layer F.Cu) (net 13))
+  (segment (start 57.26 54.61) (end 57.785 55.135) (width 0.508) (layer F.Cu) (net 13))
+  (segment (start 55.372 54.61) (end 55.372 53.172) (width 0.508) (layer F.Cu) (net 13))
+  (segment (start 55.245 53.045) (end 55.245 51.689) (width 0.508) (layer F.Cu) (net 13))
+  (segment (start 55.372 53.172) (end 55.245 53.045) (width 0.508) (layer F.Cu) (net 13))
+  (segment (start 53.848 54.61) (end 53.848 57.785) (width 0.508) (layer F.Cu) (net 14))
+  (segment (start 53.848 54.61) (end 53.848 53.002) (width 0.508) (layer F.Cu) (net 14))
+  (segment (start 53.975 52.875) (end 53.975 51.689) (width 0.508) (layer F.Cu) (net 14))
+  (segment (start 53.848 53.002) (end 53.975 52.875) (width 0.508) (layer F.Cu) (net 14))
+  (segment (start 61.722 53.975) (end 61.722 51.816) (width 0.508) (layer F.Cu) (net 15))
+  (segment (start 61.722 51.816) (end 61.595 51.689) (width 0.508) (layer F.Cu) (net 15))
   (zone (net 3) (net_name GND) (layer F.Cu) (hatch edge 0.508)
     (connect_pads (clearance 0.762))

Commit message: Routed PCB
Parts:
- moved RP1 0.97 mm to (49.8, 46.6)
Routing:
- net +5V: track 0.00 -> 92.4 mm
- net vgnd: track 0.00 -> 66.3 mm, vias 0 -> 1
- net GND: track 13.9 -> 78.0 mm, vias 0 -> 1
- net N-000023: track 0.00 -> 25.0 mm, vias 0 -> 1
- net N-000025: track 2.34 -> 25.2 mm
- net AREF: track 0.00 -> 19.3 mm
- net out: track 2.34 -> 17.7 mm
- net N-000026: track 8.76 -> 7.69 mm
- added copper zone on B.Cu, net vgnd
- added copper zone on F.Cu, net vgnd
- removed copper zone on B.Cu, net GND
- removed copper zone on F.Cu, net GND
Other:
- net class Default: clearance 0.254 -> 0.2032
- rule trace_clearance: 0.254 -> 0.2032
